File: pic24f16ka102_board.kicad_sch (KiCad schematic)
At the start: 52 parts, among them IC1 PIC24F16KA102-I_SS, J1 Jack-DC, J2 USB_B_Micro, J3 Conn_01x09_Socket, J4 Conn_01x09_Socket, J5 Conn_01x06_Pin, J6 Drive0, J7 Drive1, J8 I2C_Conn, J9 I2C_Conn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

Commit message: fix
Parts:
- removed C9: C, symbol Device:C
- removed D4, D6: D, symbol Device:D
- removed J6: Drive0, symbol Connector:Conn_01x02_Socket
- removed J7: Drive1, symbol Connector:Conn_01x02_Socket
- removed Q1, Q2: NMOS, symbol Simulation_SPICE:NMOS
- removed R12, R8: R, symbol Device:R
- added C10, C12, C13, C14, C15, C16, C17: C, symbol Device:C
- added J10: RS485_Conn, symbol Connector:Conn_01x04_Socket
- added J6, J7: Conn_01x09_Pin, symbol Connector:Conn_01x09_Pin
- added R13: 120, symbol Device:R
- J5: value Conn_01x06_Pin -> PICWr_Conn
- renumbered C10 to C9, D7 to D4, R13 to R11, R14 to R12, R9 to R8, R11 to R9
Connections:
- net +3V3: now also J8.2 (Pin_2), J9.2 (Pin_2), C12.1, C13.1, C16.1, C17.1
- net +5V: now also U2.14 (~{RESET})
- net AN0: now also J6.1 (Pin_1)
- net AN10: now also J6.7 (Pin_7)
- net AN11: now also J6.8 (Pin_8)
- net AN12: now also J6.9 (Pin_9)
- net AN2: now also J6.3 (Pin_3)
- net AN3: now also J6.4 (Pin_4)
- net AN5: now also J6.6 (Pin_6)
- net GND: now also C12.2, C13.2, C16.2, C17.2
- net RB10: now also J7.3 (Pin_3)
- net RB11: now also J7.2 (Pin_2)
- net RB15: now also J7.1 (Pin_1)
- net RB4: now also J7.9 (Pin_9)
- net RB6: now also J7.7 (Pin_7)
- net RX1: now also J6.5 (Pin_5)
- net SCL: now also J7.5 (Pin_5)
- net SDA: now also J7.8 (Pin_8)
- net TX1: now also J7.6 (Pin_6)
- net VCC: no longer C11.1, J8.2 (Pin_2), J9.2 (Pin_2)
- net ~{RTS1}: now also J7.4 (Pin_4)
- net at R8.2, SW3.2: now also IC1.19 (IC1/CN9/RA7); no longer IC1.20 (OC1/C2OUT/INT2/CTED1/CN8/RA6)
- net at IC1.1 (~{MCLR}/VPP/RA5), R7.2: no longer U2.14 (~{RESET})
- net GND2: now reaches U4.11 (GND2)
- net GND2: now also C11.2, U4.14 (GND2), U4.16 (GND2), U4.20 (GND2), C10.2, C14.2, C15.2, J10.4 (Pin_4)
- net at U4.12 (Visoout), U4.19 (Visoin): now also C11.1, C10.1, C14.1, C15.1, J10.1 (Pin_1)
- net at U4.13 (Y): now also U4.18 (A), J10.2 (Pin_2), R13.1
- net at U4.15 (Z): now also U4.17 (B), J10.3 (Pin_3), R13.2
- net at R10.1: now also IC1.20 (OC1/C2OUT/INT2/CTED1/CN8/RA6); no longer IC1.19 (IC1/CN9/RA7)
- net DRIVE0 renamed AN1
- net AN1: now also J6.2 (Pin_2)
Other:
- moved on the sheet: C8, J5, J8, J9, R11, R12, U3
